File: pcb/boot_main/app_flash.kicad_sch (KiCad schematic)
At the start: 4 parts, among them U5 W25Q32JVSS

Commit message: Assign footprints
Parts:
- C18: footprint (none) -> Capacitor_SMD:C_0603_1608Metric
- R33, R34: footprint (none) -> Resistor_SMD:R_0603_1608Metric
Changed lines of the file:
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@@
 			)
 		)
-		(property "Footprint" ""
+		(property "Footprint" "Resistor_SMD:R_0603_1608Metric"
 			(at 134.62 109.728 90)
 			(effects
@@
 			)
 		)
-		(property "Footprint" ""
+		(property "Footprint" "Capacitor_SMD:C_0603_1608Metric"
 			(at 160.9852 85.09 0)
 			(effects
@@
 			)
 		)
-		(property "Footprint" ""
+		(property "Footprint" "Resistor_SMD:R_0603_1608Metric"
 			(at 121.92 104.648 90)
 			(effects
