File: pcb/boot_main/cap_sense.kicad_sch (KiCad schematic)
At the start: 14 parts, among them J1 Conn_01x10_Pin, U4 AT42QT1070-M

Commit message: Assign footprints
Parts:
- C4: footprint (none) -> Capacitor_SMD:C_0603_1608Metric
- J1: footprint (none) -> Connector_PinHeader_2.54mm:PinHeader_1x10_P2.54mm_Vertical
- R10, R11, R12, R3, R32, R4, R5, R6, R7, R8, R9: footprint (none) -> Resistor_SMD:R_0603_1608Metric
Changed lines of the file:
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@@
 			)
 		)
-		(property "Footprint" ""
+		(property "Footprint" "Resistor_SMD:R_0603_1608Metric"
 			(at 175.26 130.048 90)
 			(effects
@@
 			)
 		)
-		(property "Footprint" ""
+		(property "Footprint" "Resistor_SMD:R_0603_1608Metric"
 			(at 104.902 87.63 90)
 			(effects
@@
 			)
 		)
-		(property "Footprint" ""
+		(property "Footprint" "Resistor_SMD:R_0603_1608Metric"
 			(at 129.032 87.63 90)
 			(effects
@@
 			)
 		)
-		(property "Footprint" ""
+		(property "Footprint" "Capacitor_SMD:C_0603_1608Metric"
 			(at 141.9352 81.28 0)
 			(effects
@@
 			)
 		)
-		(property "Footprint" ""
+		(property "Footprint" "Resistor_SMD:R_0603_1608Metric"
 			(at 175.26 98.298 90)
 			(effects
@@
 			)
 		)
-		(property "Footprint" ""
+		(property "Footprint" "Resistor_SMD:R_0603_1608Metric"
 			(at 175.26 136.398 90)
 			(effects
@@
 			)
 		)
-		(property "Footprint" ""
+		(property "Footprint" "Resistor_SMD:R_0603_1608Metric"
 			(at 175.26 117.348 90)
 			(effects
@@
 			)
 		)
-		(property "Footprint" ""
+		(property "Footprint" "Resistor_SMD:R_0603_1608Metric"
 			(at 175.26 123.698 90)
 			(effects
@@
 			)
 		)
-		(property "Footprint" ""
+		(property "Footprint" "Resistor_SMD:R_0603_1608Metric"
 			(at 112.522 87.63 90)
 			(effects
@@
 			)
 		)
-		(property "Footprint" ""
+		(property "Footprint" "Connector_PinHeader_2.54mm:PinHeader_1x10_P2.54mm_Vertical"
 			(at 220.98 116.84 0)
 			(effects
@@
 			)
 		)
-		(property "Footprint" ""
+		(property "Footprint" "Resistor_SMD:R_0603_1608Metric"
 			(at 121.412 87.63 90)
 			(effects
@@
 			)
 		)
-		(property "Footprint" ""
+		(property "Footprint" "Resistor_SMD:R_0603_1608Metric"
 			(at 175.26 110.998 90)
 			(effects
@@
 			)
 		)
-		(property "Footprint" ""
+		(property "Footprint" "Resistor_SMD:R_0603_1608Metric"
 			(at 175.26 104.648 90)
 			(effects

Commit message: push parts around
Parts:
- R10, R11, R12, R32, R7, R8, R9: footprint Resistor_SMD:R_0603_1608Metric -> Resistor_SMD:R_0402_1005Metric
Changed lines of the file:
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@@
 			)
 		)
-		(property "Footprint" "Resistor_SMD:R_0603_1608Metric"
+		(property "Footprint" "Resistor_SMD:R_0402_1005Metric"
 			(at 175.26 130.048 90)
 			(effects
@@
 			)
 		)
-		(property "Footprint" "Resistor_SMD:R_0603_1608Metric"
+		(property "Footprint" "Resistor_SMD:R_0402_1005Metric"
 			(at 175.26 98.298 90)
 			(effects
@@
 			)
 		)
-		(property "Footprint" "Resistor_SMD:R_0603_1608Metric"
+		(property "Footprint" "Resistor_SMD:R_0402_1005Metric"
 			(at 175.26 136.398 90)
 			(effects
@@
 			)
 		)
-		(property "Footprint" "Resistor_SMD:R_0603_1608Metric"
+		(property "Footprint" "Resistor_SMD:R_0402_1005Metric"
 			(at 175.26 117.348 90)
 			(effects
@@
 			)
 		)
-		(property "Footprint" "Resistor_SMD:R_0603_1608Metric"
+		(property "Footprint" "Resistor_SMD:R_0402_1005Metric"
 			(at 175.26 123.698 90)
 			(effects
@@
 			)
 		)
-		(property "Footprint" "Resistor_SMD:R_0603_1608Metric"
+		(property "Footprint" "Resistor_SMD:R_0402_1005Metric"
 			(at 175.26 110.998 90)
 			(effects
@@
 			)
 		)
-		(property "Footprint" "Resistor_SMD:R_0603_1608Metric"
+		(property "Footprint" "Resistor_SMD:R_0402_1005Metric"
 			(at 175.26 104.648 90)
 			(effects

Commit message: Some initial layout
Other:
- note added: "TODO: See if I can remove these and configure pull-ups on rpi"
Changed lines of the file:
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@@
+		)
+	)
+	(rectangle
+		(start 104.14 62.23)
+		(end 137.16 93.98)
+		(stroke
+			(width 0)
+			(type default)
+		)
+		(fill
+			(type none)
+		)
+	)
+	(text "TODO: See if I can remove these \nand configure pull-ups on rpi"
+		(exclude_from_sim no)
+		(at 121.158 65.024 0)
+		(effects
+			(font
+				(size 1.27 1.27)
+			)
 		)
 	)

Commit message: MOre layout
Parts:
- J1: footprint Connector_PinHeader_2.54mm:PinHeader_1x10_P2.54mm_Vertical -> Connector_FFC-FPC:Hirose_FH12-10S-0.5SH_1x10-1MP_P0.50mm_Horizontal
Connections:
- net GUARD: now also J1.9 (Pin_9); no longer J1.3 (Pin_3)
- net KEY1: now also J1.8 (Pin_8); no longer J1.4 (Pin_4)
- net KEY2: now also J1.7 (Pin_7); no longer J1.5 (Pin_5)
- net KEY4: now also J1.5 (Pin_5); no longer J1.7 (Pin_7)
- net KEY5: now also J1.4 (Pin_4); no longer J1.8 (Pin_8)
- net KEY6: now also J1.3 (Pin_3); no longer J1.9 (Pin_9)
Other:
- moved on the sheet: J1
Changed lines of the file:
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@@
+	(wire
+		(pts
+			(xy 212.09 124.46) (xy 217.17 124.46)
+		)
+		(stroke
+			(width 0)
+			(type default)
+		)
+	)
 	(wire
 		(pts
@@
 	(wire
 		(pts
+			(xy 213.36 127) (xy 217.17 127)
+		)
+		(stroke
+			(width 0)
+			(type default)
+		)
+	)
+	(wire
+		(pts
 			(xy 130.81 96.52) (xy 132.08 96.52)
 		)
@@
 	(wire
 		(pts
-			(xy 209.55 116.84) (xy 215.9 116.84)
-		)
-		(stroke
-			(width 0)
-			(type default)
-		)
-	)
-	(wire
-		(pts
-			(xy 213.36 127) (xy 215.9 127)
-		)
-		(stroke
-			(width 0)
-			(type default)
-		)
-	)
-	(wire
-		(pts
-			(xy 226.06 110.49) (xy 226.06 114.3)
+			(xy 212.09 111.76) (xy 217.17 111.76)
+		)
+		(stroke
+			(width 0)
+			(type default)
+		)
+	)
+	(wire
+		(pts
+			(xy 226.06 110.49) (xy 217.17 110.49)
 		)
 		(stroke
@@
 	(wire
 		(pts
+			(xy 217.17 132.08) (xy 217.17 139.7)
+		)
+		(stroke
+			(width 0)
+			(type default)
+		)
+	)
+	(wire
+		(pts
 			(xy 179.07 115.57) (xy 208.28 115.57)
 		)
@@
 	(wire
 		(pts
+			(xy 179.07 121.92) (xy 217.17 121.92)
+		)
+		(stroke
+			(width 0)
+			(type default)
+		)
+	)
+	(wire
+		(pts
 			(xy 147.32 88.9) (xy 147.32 73.66)
 		)
@@
 	(wire
 		(pts
+			(xy 217.17 110.49) (xy 217.17 109.22)
+		)
+		(stroke
+			(width 0)
+			(type default)
+		)
+	)
+	(wire
+		(pts
 			(xy 165.1 111.76) (xy 165.1 134.62)
 		)
@@
 	(wire
 		(pts
-			(xy 215.9 110.49) (xy 226.06 110.49)
+			(xy 224.79 130.81) (xy 217.17 130.81)
 		)
 		(stroke
@@
 	(wire
 		(pts
-			(xy 215.9 109.22) (xy 215.9 110.49)
+			(xy 208.28 119.38) (xy 217.17 119.38)
 		)
 		(stroke
@@
 	(wire
 		(pts
-			(xy 215.9 129.54) (xy 215.9 138.43)
+			(xy 214.63 139.7) (xy 217.17 139.7)
 		)
 		(stroke
@@
 	(wire
 		(pts
+			(xy 209.55 116.84) (xy 217.17 116.84)
+		)
+		(stroke
+			(width 0)
+			(type default)
+		)
+	)
+	(wire
+		(pts
 			(xy 132.08 111.76) (xy 132.08 119.38)
 		)
@@
 	(wire
 		(pts
-			(xy 212.09 124.46) (xy 215.9 124.46)
+			(xy 217.17 130.81) (xy 217.17 129.54)
+		)
+		(stroke
+			(width 0)
+			(type default)
+		)
+	)
+	(wire
+		(pts
+			(xy 210.82 114.3) (xy 217.17 114.3)
 		)
 		(stroke
@@
 	(wire
 		(pts
-			(xy 212.09 111.76) (xy 215.9 111.76)
-		)
-		(stroke
-			(width 0)
-			(type default)
-		)
-	)
-	(wire
-		(pts
 			(xy 166.37 109.22) (xy 166.37 128.27)
 		)
@@
 	(wire
 		(pts
-			(xy 210.82 114.3) (xy 215.9 114.3)
-		)
-		(stroke
-			(width 0)
-			(type default)
-		)
-	)
-	(wire
-		(pts
 			(xy 179.07 128.27) (xy 212.09 128.27)
 		)
@@
 	(wire
 		(pts
-			(xy 179.07 121.92) (xy 215.9 121.92)
-		)
-		(stroke
-			(width 0)
-			(type default)
-		)
-	)
-	(wire
-		(pts
-			(xy 208.28 119.38) (xy 215.9 119.38)
-		)
-		(stroke
-			(width 0)
-			(type default)
-		)
-	)
-	(wire
-		(pts
 			(xy 147.32 119.38) (xy 147.32 121.92)
 		)
@@
 		(pts
 			(xy 167.64 106.68) (xy 167.64 121.92)
-		)
-		(stroke
-			(width 0)
-			(type default)
-		)
-	)
-	(wire
-		(pts
-			(xy 215.9 101.6) (xy 215.9 106.68)
 		)
 		(stroke
@@
 	(symbol
 		(lib_id "power:GND")
-		(at 215.9 138.43 0)
+		(at 226.06 110.49 0)
+		(mirror y)
 		(unit 1)
 		(exclude_from_sim no)
@@
 		(fields_autoplaced yes)
 		(property "Reference" "#PWR030"
-			(at 215.9 144.78 0)
+			(at 226.06 116.84 0)
 			(effects
 				(font
@@
 		)
 		(property "Value" "GND"
-			(at 215.9 143.51 0)
-			(effects
-				(font
-					(size 1.27 1.27)
-				)
+			(at 228.6 111.7599 0)
+			(effects
+				(font
+					(size 1.27 1.27)
+				)
+				(justify right)
 			)
 		)
 		(property "Footprint" ""
-			(at 215.9 138.43 0)
+			(at 226.06 110.49 0)
 			(effects
 				(font
@@
 		)
 		(property "Datasheet" ""
-			(at 215.9 138.43 0)
+			(at 226.06 110.49 0)
 			(effects
 				(font
@@
 		)
 		(property "Description" "Power symbol creates a global label with name \"GND\" , ground"
-			(at 215.9 138.43 0)
+			(at 226.06 110.49 0)
 			(effects
 				(font
@@
 	(symbol
 		(lib_id "power:+3V3")
-		(at 215.9 101.6 0)
+		(at 214.63 139.7 0)
+		(mirror y)
 		(unit 1)
 		(exclude_from_sim no)
@@
 		(fields_autoplaced yes)
 		(property "Reference" "#PWR017"
-			(at 215.9 105.41 0)
+			(at 214.63 143.51 0)
 			(effects
 				(font
@@
 		)
 		(property "Value" "+3V3"
-			(at 215.9 96.52 0)
-			(effects
-				(font
-					(size 1.27 1.27)
-				)
+			(at 217.17 138.4299 0)
+			(effects
+				(font
+					(size 1.27 1.27)
+				)
+				(justify right)
 			)
 		)
 		(property "Footprint" ""
-			(at 215.9 101.6 0)
+			(at 214.63 139.7 0)
 			(effects
 				(font
@@
 		)
 		(property "Datasheet" ""
-			(at 215.9 101.6 0)
+			(at 214.63 139.7 0)
 			(effects
 				(font
@@
 		)
 		(property "Description" "Power symbol creates a global label with name \"+3V3\""
-			(at 215.9 101.6 0)
+			(at 214.63 139.7 0)
 			(effects
 				(font
@@
 	(symbol
 		(lib_id "Connector:Conn_01x10_Pin")
-		(at 220.98 116.84 0)
-		(mirror y)
+		(at 222.25 121.92 180)
 		(unit 1)
 		(exclude_from_sim no)
@@
 		(dnp no)
 		(property "Reference" "J1"
-			(at 220.345 101.6 0)
+			(at 221.615 137.16 0)
 			(effects
 				(font
@@
 		)
 		(property "Value" "Conn_01x10_Pin"
-			(at 220.345 104.14 0)
-			(effects
-				(font
-					(size 1.27 1.27)
-				)
-			)
-		)
-		(property "Footprint" "Connector_PinHeader_2.54mm:PinHeader_1x10_P2.54mm_Vertical"
-			(at 220.98 116.84 0)
+			(at 221.615 134.62 0)
+			(effects
+				(font
+					(size 1.27 1.27)
+				)
+			)
+		)
+		(property "Footprint" "Connector_FFC-FPC:Hirose_FH12-10S-0.5SH_1x10-1MP_P0.50mm_Horizontal"
+			(at 222.25 121.92 0)
 			(effects
 				(font
@@
 		)
 		(property "Datasheet" "~"
-			(at 220.98 116.84 0)
+			(at 222.25 121.92 0)
 			(effects
 				(font
@@
 		)
 		(property "Description" "Generic connector, single row, 01x10, script generated"
-			(at 220.98 116.84 0)
+			(at 222.25 121.92 0)
 			(effects
 				(font
@@
 	(symbol
 		(lib_id "power:GND")
-		(at 226.06 114.3 0)
+		(at 224.79 130.81 0)
+		(mirror y)
 		(unit 1)
 		(exclude_from_sim no)
@@
 		(fields_autoplaced yes)
 		(property "Reference" "#PWR018"
-			(at 226.06 120.65 0)
+			(at 224.79 137.16 0)
 			(effects
 				(font
@@
 		)
 		(property "Value" "GND"
-			(at 226.06 119.38 0)
-			(effects
-				(font
-					(size 1.27 1.27)
-				)
+			(at 227.33 132.0799 0)
+			(effects
+				(font
+					(size 1.27 1.27)
+				)
+				(justify right)
 			)
 		)
 		(property "Footprint" ""
-			(at 226.06 114.3 0)
+			(at 224.79 130.81 0)
 			(effects
 				(font
@@
 		)
 		(property "Datasheet" ""
-			(at 226.06 114.3 0)
+			(at 224.79 130.81 0)
 			(effects
 				(font
@@
 		)
 		(property "Description" "Power symbol creates a global label with name \"GND\" , ground"
-			(at 226.06 114.3 0)
-			(effects
-				(font
+			(at 224.79 130.81 0)
+			(effects
+				(font

Commit message: move cap sense ic to front panel
Parts:
- removed C4: 0.1u, Capacitor_SMD:C_0603_1608Metric, symbol Device:C
- removed J1: Conn_01x10_Pin, Connector_FFC-FPC:Hirose_FH12-10S-0.5SH_1x10-1MP_P0.50mm_Horizontal, symbol Connector:Conn_01x10_Pin
- removed R10, R11, R12, R32, R7, R8, R9: 10k, Resistor_SMD:R_0402_1005Metric, symbol Device:R
- removed R3, R4: 10k, Resistor_SMD:R_0603_1608Metric, symbol Device:R
- removed R5, R6: 4.7k, Resistor_SMD:R_0603_1608Metric, symbol Device:R
- removed U4: AT42QT1070-M, Package_DFN_QFN:VQFN-20-1EP_3x3mm_P0.45mm_EP1.55x1.55mm, symbol Sensor_Touch:AT42QT1070-M
Other:
- note removed: "TODO: See if I can remove these and configure pull-ups on rpi"
