File: pcb/boot_main/boot_main.kicad_sch (KiCad schematic)
At the start: 36 parts, among them J1 Conn_01x06_Pin, J2 Conn_01x02_Pin, P1 USB_C_Plug_USB2.0, SW1 SW_Push, SW2 SW_Push, U1 RP2040, U2 NCP1117-3.3_SOT223, U3 W25Q32JVZP, Y1 Crystal_GND24

Commit message: More layout
Connections:
- net +3V3: now also R35.2; no longer R35.1, U1.26 (RUN)
- net B2_LIGHT: now also U1.2 (GPIO0); no longer U1.31 (GPIO20)
- net B3_LIGHT: now also U1.8 (GPIO6); no longer U1.34 (GPIO22)
- net RUN: now reaches SW2.1
- net RUN: now also R35.1, U1.26 (RUN); no longer R35.2
Other:
- note removed: "TODO: Maybe change from buttons to pins?"
- moved on the sheet: R35
Changed lines of the file:
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@@
 	)
 	(junction
-		(at 228.6 33.02)
-		(diameter 0)
-		(color 0 0 0 0)
-	)
-	(junction
 		(at 41.91 102.87)
 		(diameter 0)
@@
 		(color 0 0 0 0)
 	)
+	(junction
+		(at 236.22 33.02)
+		(diameter 0)
+		(color 0 0 0 0)
+	)
 	(wire
 		(pts
@@
 	(wire
 		(pts
-			(xy 238.76 33.02) (xy 248.92 33.02)
-		)
-		(stroke
-			(width 0)
-			(type default)
-		)
-	)
-	(wire
-		(pts
 			(xy 143.51 81.28) (xy 143.51 87.63)
 		)
@@
 	(wire
 		(pts
-			(xy 228.6 24.13) (xy 228.6 33.02)
-		)
-		(stroke
-			(width 0)
-			(type default)
-		)
-	)
-	(wire
-		(pts
 			(xy 138.43 182.88) (xy 138.43 185.42)
 		)
@@
 	(wire
 		(pts
+			(xy 236.22 31.75) (xy 236.22 33.02)
+		)
+		(stroke
+			(width 0)
+			(type default)
+		)
+	)
+	(wire
+		(pts
 			(xy 140.97 81.28) (xy 143.51 81.28)
 		)
@@
 	(wire
 		(pts
-			(xy 228.6 33.02) (xy 231.14 33.02)
-		)
-		(stroke
-			(width 0)
-			(type default)
-		)
-	)
-	(wire
-		(pts
 			(xy 208.28 105.41) (xy 215.9 105.41)
 		)
@@
 	(wire
 		(pts
+			(xy 236.22 33.02) (xy 248.92 33.02)
+		)
+		(stroke
+			(width 0)
+			(type default)
+		)
+	)
+	(wire
+		(pts
 			(xy 208.28 152.4) (xy 217.17 152.4)
 		)
@@
 	(wire
 		(pts
+			(xy 236.22 21.59) (xy 236.22 24.13)
+		)
+		(stroke
+			(width 0)
+			(type default)
+		)
+	)
+	(wire
+		(pts
 			(xy 125.73 72.39) (xy 125.73 73.66)
 		)
@@
 	(wire
 		(pts
-			(xy 163.83 151.13) (xy 173.99 151.13)
+			(xy 163.83 110.49) (xy 173.99 110.49)
 		)
 		(stroke
@@
 	(wire
 		(pts
-			(xy 222.25 33.02) (xy 228.6 33.02)
+			(xy 229.87 33.02) (xy 236.22 33.02)
 		)
 		(stroke
@@
 	(wire
 		(pts
-			(xy 163.83 146.05) (xy 173.99 146.05)
+			(xy 163.83 95.25) (xy 173.99 95.25)
 		)
 		(stroke
@@
 		)
 	)
-	(rectangle
-		(start 138.43 15.24)
-		(end 269.24 44.45)
-		(stroke
-			(width 0)
-			(type default)
-		)
-		(fill
-			(type none)
-		)
-	)
 	(text "BOOTSEL button forces entry to bootloader\nby breaking SPI flash communication at boot"
 		(exclude_from_sim no)
@@
 	(text "Reset mechanism via button"
 		(exclude_from_sim no)
-		(at 248.666 20.32 0)
+		(at 253.238 21.082 0)
 		(effects
 			(font
@@
 		)
 	)
-	(text "TODO: Maybe change from \nbuttons to pins?"
-		(exclude_from_sim no)
-		(at 206.248 27.94 0)
-		(effects
-			(font
-				(size 1.27 1.27)
-			)
-		)
-	)
 	(label "B2_LIGHT"
-		(at 165.1 146.05 0)
+		(at 165.1 95.25 0)
 		(fields_autoplaced yes)
 		(effects
@@
 	)
 	(label "B3_LIGHT"
-		(at 165.1 151.13 0)
+		(at 165.1 110.49 0)
 		(fields_autoplaced yes)
 		(effects
@@
 	)
 	(label "RUN"
-		(at 222.25 33.02 0)
+		(at 229.87 33.02 0)
 		(fields_autoplaced yes)
 		(effects
@@
 	(symbol
 		(lib_id "power:+3V3")
-		(at 228.6 24.13 0)
+		(at 236.22 21.59 0)
 		(unit 1)
 		(exclude_from_sim no)
@@
 		(fields_autoplaced yes)
 		(property "Reference" "#PWR042"
-			(at 228.6 27.94 0)
+			(at 236.22 25.4 0)
 			(effects
 				(font
@@
 		)
 		(property "Value" "+3V3"
-			(at 228.6 19.05 0)
+			(at 236.22 16.51 0)
 			(effects
 				(font
@@
 		)
 		(property "Footprint" ""
-			(at 228.6 24.13 0)
+			(at 236.22 21.59 0)
 			(effects
 				(font
@@
 		)
 		(property "Datasheet" ""
-			(at 228.6 24.13 0)
+			(at 236.22 21.59 0)
 			(effects
 				(font
@@
 		)
 		(property "Description" "Power symbol creates a global label with name \"+3V3\""
-			(at 228.6 24.13 0)
+			(at 236.22 21.59 0)
 			(effects
 				(font
@@
 	(symbol
 		(lib_id "Device:R")
-		(at 234.95 33.02 90)
+		(at 236.22 27.94 180)
 		(unit 1)
 		(exclude_from_sim no)
@@
 		(fields_autoplaced yes)
 		(property "Reference" "R35"
-			(at 234.95 26.67 90)
+			(at 238.76 26.6699 0)
 			(effects
 				(font
 					(size 1.27 1.27)
 				)
+				(justify right)
 			)
 		)
 		(property "Value" "10k"
-			(at 234.95 29.21 90)
+			(at 238.76 29.2099 0)
 			(effects
 				(font
 					(size 1.27 1.27)
 				)
+				(justify right)
 			)
 		)
 		(property "Footprint" "Resistor_SMD:R_0603_1608Metric"
-			(at 234.95 34.798 90)
+			(at 237.998 27.94 90)
 			(effects
 				(font
@@
 		)
 		(property "Datasheet" "~"
-			(at 234.95 33.02 0)
+			(at 236.22 27.94 0)
 			(effects
 				(font
@@
 		)
 		(property "Description" "Resistor"
-			(at 234.95 33.02 0)
+			(at 236.22 27.94 0)
 			(effects
 				(font
